Commit message: upload tm_900(rviz,gazebo,moveit) with arm,camera

File: tm_ws18_900/src/tmr_ros1-master/tm5_description/urdf/tm5_900_robot.urdf.xacro (robot description, xacro)
@@ -2,5 +2,5 @@
 <robot xmlns:xacro="http://wiki.ros.org/xacro" name="tm5_900" >
   <!--xacro:arg name="transmission_hw_interface" default="hardware_interface/PositionJointInterface"/-->
-  <!--xacro:arg name="stl_mesh" default="false"/-->
+  <xacro:arg name="stl_mesh" default="false"/>
   <xacro:arg name="prefix" default="" />
   <xacro:arg name="gripper" default="robotiq_2f" />
@@ -17,4 +17,8 @@
     <xacro:robotiq_2f prefix="$(arg prefix)"/>
   </xacro:if>
+  <xacro:include filename="$(find realsense_ros_gazebo)/xacro/depthcam.xacro"/>
+  <xacro:realsense_d435 sensor_name="d435" parent_link="tool0" rate="10">
+  <origin rpy="-0.00095 -1.57 -1.57" xyz="-0.00006286 0.105 0.0376066"/>
+  </xacro:realsense_d435>
   <link name="world" />
   <joint name="world_joint" type="fixed">

File: tm_ws18_900/src/tmr_ros1-master/tmr_description/xacro/gripper/robotiq_2f.urdf.xacro (robot description, xacro)
@@ -28,4 +28,9 @@
     <child link="robotiq_coupler"/>
   </joint>
+  <!-- <joint name="robotiq_coupler_joint" type="fixed">
+    <origin xyz="0 0 0.004" rpy="0 0 ${-pi/2.0}" />
+    <parent link="${prefix}flange_link"/>
+    <child link="robotiq_coupler"/>
+  </joint> -->
   <gazebo reference="robotiq_coupler">
     <mu1>0.9</mu1>
@@ -44,4 +49,7 @@
     <origin xyz="0 0 0.004" rpy="0 ${-pi/2} ${pi}"/>
   </xacro:robotiq_85_gripper>
+  <!-- <xacro:robotiq_85_gripper prefix="" parent="robotiq_coupler" >
+    <origin xyz="0 0 0.004" rpy="0 ${-pi/2} ${pi}"/>
+  </xacro:robotiq_85_gripper>  -->
   <gazebo>
     <gripper name="gazebo_gripper">
